File: RetroNES.sch (EAGLE design)
At the start: 8 parts, among them IC1 ATMEGA32U4-AU

Commit message: First commit
Parts:
- removed CN1: (no value), adafruit:USBMINIB
- removed IC1: ATMEGA32U4-AU, adafruit:ATMEGA32U4-AU
- removed NES: NES_SOCKET, RetroNES:NES_SOCKET
- added A-BUTTON, B-BUTTON, X-BUTTON, Y-BUTTON: AB, NES:AB
- added C2: 8pf, adafruit:C-USC0402
- added C3: 8pF, adafruit:C-USC0402
- added DOWN-BUTTON, LEFT-BUTTON, RIGHT-BUTTON, SELECT-BUTTON, START-BUTTON, UP-BUTTON: DPAD-SS, NES:DPAD-SS
- added L, R: (no value), pinhead:PINHD-1X2
- added R10, R11, R12, R3, R4, R5, R6, R7, R8, R9: 1k, adafruit:R-US_R0402
- added U$1: ATMEGA32U41:1-LESS_PASTE, SparkFun-DigitalIC:ATMEGA32U41:1-LESS_PASTE
- added U$2: CX2520DB, adamtemp:CX2520DB
- C1: device adafruit:C-USC0805 -> adafruit:C-USC0402
- R1, R2: value 22 -> 1k; device adafruit:R-US_R0805 -> adafruit:R-US_R0402
Connections:
- removed net CLOCK: IC1.PF5(ADC5/TMS), NES.CLOCK
- removed net D+: CN1.D+, R1.1
- removed net D+U: IC1.D+, R1.2
- removed net D-: CN1.D-, R2.1
- removed net D-U: IC1.D-, R2.2
- removed net DO: IC1.PF7(ADC7(TDI), NES.DO
- removed net LATCH: IC1.PF6(ADC6/TDO), NES.LATCH
- new net L: L.1, R11.1, U$1.PC6
- new net R: R.1, R12.1, U$1.PC7
- new net X: R2.1, U$1.PB6(ADC13), X-BUTTON.1
- new net XTAL1: C3.1, U$1.XTAL1, U$2.1
- new net XTAL2: C2.1, U$1.XTAL2, U$2.3
- new net Y: R1.1, U$1.PB7, Y-BUTTON.1
- net A: now also A-BUTTON.1, R10.1, U$1.PB5(ADC12); no longer IC1.PB5(OC1A/OC4B/ADC12), NES.A
- net B: now also B-BUTTON.1, R9.1, U$1.PB4(ADC11); no longer IC1.PB4(ADC11), NES.B
- net DOWN: now also DOWN-BUTTON.1, R5.1, U$1.PD4(ADC8); no longer IC1.PD4(ICP1/ADC8), NES.DOWN
- net GND: now also A-BUTTON.2, B-BUTTON.2, C2.2, C3.2, DOWN-BUTTON.2, L.2, LEFT-BUTTON.2, R.2, RIGHT-BUTTON.2, SELECT-BUTTON.2, START-BUTTON.2, U$1.GND@15, U$1.GND@23, U$1.GND@35, U$1.GND@43, U$1.PE2/!HWB, U$1.UGND, U$2.2, UP-BUTTON.2, X-BUTTON.2, Y-BUTTON.2; no longer CN1.GND, IC1.GND, IC1.GND1, IC1.GND2, IC1.GND3, IC1.PE2(HWB), IC1.UGND, NES.GND, NES.GND2
- net LEFT: now also LEFT-BUTTON.1, R6.1, U$1.PD3(TX); no longer IC1.PD3(INT3/TXD1), NES.LEFT
- net MISO: now also U$1.PB3(MISO); no longer IC1.PB3(PDO/MISO)
- net MOSI: now also U$1.PB2(MOSI); no longer IC1.PB2(PDI/MISO)
- net RESET: now also U$1.!RESET; no longer IC1./RESET
- net RIGHT: now also R4.1, RIGHT-BUTTON.1, U$1.PD2(RX); no longer IC1.PD2(INT2/RXD1), NES.RIGHT
- net SCK: now also U$1.PB1(SCK); no longer IC1.PB1(SCK)
- net SCL: now also U$1.PD0(SCL); no longer IC1.PD0(INT0/OC0B)
- net SDA: now also U$1.PD1(SDA); no longer IC1.PD1(INT1/SDA)
- net SELECT: now also R7.1, SELECT-BUTTON.1, U$1.PD7(ADC10); no longer IC1.PD7(OC4D/ADC10/T0), NES.SELECT
- net START: now also R8.1, START-BUTTON.1, U$1.PD6(ADC9); no longer IC1.PD6(T1/OC4D/ADC9), NES.START
- net UCAP: now also U$1.UCAP; no longer IC1.UCAP
- net UP: now also R3.1, U$1.PD5, UP-BUTTON.1; no longer IC1.PD5(XCK/CTS), NES.UP
- net VCC: now also R1.2, R10.2, R11.2, R12.2, R2.2, R3.2, R4.2, R5.2, R6.2, R7.2, R8.2, R9.2, U$1.AREF, U$1.AVCC@24, U$1.AVCC@44, U$1.UVCC, U$1.VCC@14, U$1.VCC@34; no longer CN1.VBUS, IC1.AREF, IC1.AVCC, IC1.AVCC1, IC1.UVCC, IC1.VCC, IC1.VCC1, NES.VCC
Other:
- moved on the sheet: R1, R2
